File: Charging.sch (KiCad schematic (older format))
At the start: 15 parts, among them K2 T9AS1D12-24, K3 T9AS1D12-24, Q2 DMN3730U, Q3 DMP10H4D2S, U8 ACHS-7122

Commit message: Add files via upload
Connections:
- net CHRG_OUT+ renamed PACK+
- net CHRG_OUT- renamed PACK-
Changed lines of the file:
@@
 CHRG_IN-
 Text HLabel 1250 1450 0    50   Input ~ 0
-CHRG_OUT+
+PACK+
 Text HLabel 1250 1550 0    50   Input ~ 0
-CHRG_OUT-
+PACK-
 Text Label 1350 1200 0    50   ~ 0
 CHRG_IN+
@@
 	1350 1200 1250 1200
 Text Label 1350 1450 0    50   ~ 0
-CHRG_OUT+
+PACK+
 Text Label 1350 1550 0    50   ~ 0
-CHRG_OUT-
+PACK-
 Wire Wire Line
 	1250 1450 1350 1450
@@
 	4950 2350 5050 2350
 Text Label 4950 2350 2    50   ~ 0
-CHRG_OUT-
+PACK-
 $Comp
 L Lafayette_Electric_Car_Internals:ACHS-7122 U8
@@
 $EndComp
 Text Label 5000 3800 2    50   ~ 0
-CHRG_OUT+
+PACK+
 $Comp
 L Device:C C12
