File: PacMan.kicad_pcb (KiCad board)
At the start: 2 copper layers, 134.6 x 109.2 mm, 169 parts, among them J1 POWER+, J10 SLOOP, J11 Panel, J2 POWER-, J3 SEG+ CellMen, J4 SEG- CellMen, J5 Charge Detection, J6 BusBar Current Sensor, J7 GLV/CAN, J8 AIR Left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

Commit message: Add files via upload
Connections:
- net /PACK_RTN renamed /RTN_TSV
- U5 pad 15: /DISP_MOSI -> /MCU/DISP_MOSI
- U5 pad 31: /TS_ACTIVE -> /MCU/TS_ACTIVE
Routing:
- added copper zone on F.Cu, net /PACK_RTN
- removed copper zone on F.Cu, net /RTN_TSV
