File: PacMan.sch (KiCad schematic (older format))
At the start: 22 parts, among them J1 POWER+, J10 SLOOP, J11 Panel, J2 POWER-, J3 SEG+ CellMen, J4 SEG- CellMen, J5 Charge Detection, J6 BusBar Current Sensor, J7 GLV/CAN, J8 AIR Left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

Commit message: Add files via upload
Connections:
- net PACK_RTN is gone; now on net RTN_TSV: F2.2
Changed lines of the file:
@@
 Text Label 9950 6000 0    50   ~ 0
 LV_RTN
-Wire Notes Line width 12 style solid
-	5100 1200 5100 500
 Text Label 4150 4300 2    50   ~ 0
 CHRG_DETECT+
@@
 Wire Wire Line
 	4250 4300 4150 4300
-Wire Wire Line
-	4150 1750 4250 1750
-Wire Wire Line
-	4250 1850 4150 1850
 Text Label 4150 4500 2    50   ~ 0
 AMPS_PWR
@@
 	2250 1750 2450 1750
 Wire Wire Line
-	4250 1350 4150 1350
-Text Label 4150 1350 2    50   ~ 0
-PACK_FUSED
-Wire Wire Line
 	2150 3850 2050 3850
 Wire Wire Line
@@
 	9150 1700 9050 1700
 Text Label 9150 2450 0    50   ~ 0
-DISP_DIN
+DISP_MOSI
 Text Label 9150 2350 0    50   ~ 0
 DISP_CLK
@@
 DISP_RST
 Text Label 9150 1950 0    50   ~ 0
-DISP_BUSY
+TS_ACTIVE
 Wire Wire Line
 	9050 2450 9150 2450
@@
 Wire Wire Line
 	9350 6200 9250 6200
-Text Label 6050 1700 0    50   ~ 0
-LV_5V
-Text Label 6050 1800 0    50   ~ 0
-LV_RTN
-Wire Wire Line
-	6050 1700 5950 1700
-Wire Wire Line
-	6050 1800 5950 1800
 Text Label 6050 3400 0    50   ~ 0
 LV_5V
@@
 Wire Wire Line
 	6050 4400 5950 4400
-Text Label 6050 1350 0    50   ~ 0
-GLV_24V
-Text Label 6050 1450 0    50   ~ 0
-GLV_RTN
-Wire Wire Line
-	6050 1350 5950 1350
-Wire Wire Line
-	6050 1450 5950 1450
-Text Label 6050 1600 0    50   ~ 0
-LV_24V
-Wire Wire Line
-	5950 1600 6050 1600
 Text Label 6050 4550 0    50   ~ 0
 ~CHRG_DETECT
@@
 Text Label 9150 1300 0    50   ~ 0
 SLOOP2
-Wire Wire Line
-	4250 2650 4150 2650
-Wire Wire Line
-	4150 2750 4250 2750
-Text Label 4150 2650 2    50   ~ 0
-9V_SEG-
-Text Label 4150 2750 2    50   ~ 0
-5V_SEG-
-Text Label 4150 2850 2    50   ~ 0
-RTN_SEG-
-Wire Wire Line
-	4150 2850 4250 2850
 $Comp
 L Connector_Generic:Conn_02x03_Odd_Even J3
@@
 Wire Wire Line
 	6050 3300 5950 3300
-Text Label 4150 1850 2    50   ~ 0
-SCL_TSV
-Text Label 4150 1750 2    50   ~ 0
-SDA_TSV
 $Sheet
 S 4250 3200 1700 750
@@
 F2 "CHRG_IN+" I L 4250 3300 50
 F3 "CHRG_IN-" I L 4250 3400 50
-F4 "CHRG_OUT+" I L 4250 3750 50
-F5 "CHRG_OUT-" I L 4250 3850 50
+F4 "PACK+" I L 4250 3750 50
+F5 "PACK-" I L 4250 3850 50
 F6 "CHRG_EN" I R 5950 3650 50
 F7 "CHRG_CURRENT" I R 5950 3750 50
@@
 Text Label 4050 7250 0    50   ~ 0
 RTN_TSV
-Wire Wire Line
-	4250 2050 4150 2050
-Wire Wire Line
-	4250 1950 4150 1950
-Text Label 4150 1950 2    50   ~ 0
-DCHRG_A1
-Text Label 4150 2050 2    50   ~ 0
-DCHRG_A2
 Text Label 2450 2450 0    50   ~ 0
-PACK_RTN
-Text Label 4150 1450 2    50   ~ 0
-PACK_RTN
-Text Label 4150 1550 2    50   ~ 0
-5V_TSV
-Text Label 4150 1650 2    50   ~ 0
 RTN_TSV
-Wire Wire Line
-	4150 1650 4250 1650
-Wire Wire Line
-	4150 1550 4250 1550
-Wire Wire Line
-	4150 1450 4250 1450
 Text Label 4150 4650 2    50   ~ 0
 5V_TSV
@@
 Text Label 3650 7850 0    50   ~ 0
 RTN_TSV
-$Sheet
-S 7750 1000 1300 1900
-U 5DC1F176
-F0 "MCU" 50
-F1 "MCU.sch" 50
-F2 "SLOOP1_IN" I R 9050 1100 50
-F3 "SLOOP1_OUT" I R 9050 1200 50
-F4 "AIRS+" I R 9050 1400 50
-F5 "AIRS-" I R 9050 1500 50
-F6 "CHRG_EN" I L 7750 1550 50
-F7 "CHRG_CURRENT" I L 7750 1750 50
-F8 "SDA_GLV" I L 7750 1900 50
-F9 "SCL_GLV" I L 7750 2000 50
-F10 "~CHRG_DETECT" I L 7750 1650 50
-F11 "CAN_H" I R 9050 1600 50
-F12 "CAN_L" I R 9050 1700 50
-F13 "LV_5V" I L 7750 1200 50
-F14 "LV_RTN" I L 7750 1400 50
-F15 "BTN_LEFT" I L 7750 2150 50
-F16 "BTN_RIGHT" I L 7750 2250 50
-F17 "BTN_UP" I L 7750 2350 50
-F18 "BTN_DOWN" I L 7750 2450 50
-F19 "BTN_CENTER" I L 7750 2550 50
-F20 "DISP_DIN" I R 9050 2450 50
-F21 "DISP_CLK" I R 9050 2350 50
-F22 "DISP_CS" I R 9050 2250 50
-F23 "DISP_DC" I R 9050 2150 50
-F24 "DISP_RST" I R 9050 2050 50
-F25 "DISP_BUSY" I R 9050 1950 50
-F26 "CAN_SHIELD" I R 9050 1800 50
-F27 "LV_3V3" I L 7750 1300 50
-F28 "SLOOP2" I R 9050 1300 50
-F29 "RST_GLV_SEG+" I L 7750 2700 50
-F30 "RST_GLV_SEG-" I L 7750 2800 50
-F31 "LV_24V" I L 7750 1100 50
-F32 "GLV_24V" I R 9050 2600 50
-F33 "GLV_RTN" I R 9050 2700 50
-$EndSheet
 Text Label 9150 2600 0    50   ~ 0
 GLV_24V
@@
 Wire Notes Line width 12 style solid
 	3750 5050 5100 5050
+NoConn ~ 9850 5400
+Wire Wire Line
+	4250 1450 4150 1450
+Text Label 4150 1450 2    50   ~ 0
+PACK_FUSED
+Wire Wire Line
+	6050 1800 5950 1800
+Wire Wire Line
+	6050 1900 5950 1900
+Wire Wire Line
+	6050 1450 5950 1450
+Wire Wire Line
+	6050 1550 5950 1550
+Wire Wire Line
+	5950 1700 6050 1700
+Wire Wire Line
+	4250 2650 4150 2650
+Wire Wire Line
+	4150 2750 4250 2750
+Text Label 4150 2650 2    50   ~ 0
+9V_SEG-
+Text Label 4150 2750 2    50   ~ 0
+5V_SEG-
+Text Label 4150 2850 2    50   ~ 0
+RTN_SEG-
+Wire Wire Line
+	4150 2850 4250 2850
 Wire Wire Line
 	4150 2450 4250 2450
@@
 9V_SEG+
 Wire Notes Line width 12 style solid
-	5100 1300 5100 2900
-Wire Notes Line width 12 style solid
 	5100 2550 3750 2550
 Wire Notes Line width 12 style solid
 	5100 2150 3750 2150
+Wire Wire Line
+	4150 1550 4250 1550
+Wire Wire Line
+	4150 1650 4250 1650
+Text Label 4150 1650 2    50   ~ 0
+RTN_TSV
+Text Label 4150 1550 2    50   ~ 0
+5V_TSV
+Text Label 4150 2050 2    50   ~ 0
+DCHRG_A2
+Text Label 4150 1950 2    50   ~ 0
+DCHRG_A1
+Wire Wire Line
+	4250 1950 4150 1950
+Wire Wire Line
+	4250 2050 4150 2050
+Text Label 4150 1750 2    50   ~ 0
+SDA_TSV
+Text Label 4150 1850 2    50   ~ 0
+SCL_TSV
+Wire Wire Line
+	4250 1850 4150 1850
+Wire Wire Line
+	4150 1750 4250 1750
+Text Label 6050 1700 0    50   ~ 0
+LV_24V
+Text Label 6050 1550 0    50   ~ 0
+GLV_RTN
+Text Label 6050 1450 0    50   ~ 0
+GLV_24V
+Text Label 6050 1900 0    50   ~ 0
+LV_RTN
+Text Label 6050 1800 0    50   ~ 0
+LV_5V
 $Sheet
-S 4250 1250 1700 1700
+S 4250 1350 1700 1600
 U 5DD31136
 F0 "Power" 50
 F1 "Power.sch" 50
-F2 "GLV_24V" I R 5950 1350 50
-F3 "GLV_RTN" I R 5950 1450 50
-F4 "LV_RTN" I R 5950 1800 50
-F5 "LV_5V" I R 5950 1700 50
-F6 "LV_24V" I R 5950 1600 50
+F2 "GLV_24V" I R 5950 1450 50
+F3 "GLV_RTN" I R 5950 1550 50
+F4 "LV_RTN" I R 5950 1900 50
+F5 "LV_5V" I R 5950 1800 50
+F6 "LV_24V" I R 5950 1700 50
 F7 "DCHRG_A1" I L 4250 1950 50
 F8 "DCHRG_A2" I L 4250 2050 50
-F9 "PACK_FUSED" I L 4250 1350 50
-F10 "PACK_RTN" I L 4250 1450 50
-F11 "SDA_TSV" I L 4250 1750 50
-F12 "SCL_TSV" I L 4250 1850 50
-F13 "9V_SEG-" I L 4250 2650 50
-F14 "RTN_SEG-" I L 4250 2850 50
-F15 "9V_SEG+" I L 4250 2250 50
-F16 "RTN_SEG+" I L 4250 2450 50
-F17 "5V_SEG-" I L 4250 2750 50
-F18 "5V_SEG+" I L 4250 2350 50
-F19 "5V_TSV" I L 4250 1550 50
-F20 "RTN_TSV" I L 4250 1650 50
+F9 "PACK_FUSED" I L 4250 1450 50
+F10 "SDA_TSV" I L 4250 1750 50
+F11 "SCL_TSV" I L 4250 1850 50
+F12 "9V_SEG-" I L 4250 2650 50
+F13 "RTN_SEG-" I L 4250 2850 50
+F14 "9V_SEG+" I L 4250 2250 50
+F15 "RTN_SEG+" I L 4250 2450 50
+F16 "5V_SEG-" I L 4250 2750 50
+F17 "5V_SEG+" I L 4250 2350 50
+F18 "5V_TSV" I L 4250 1550 50
+F19 "RTN_TSV" I L 4250 1650 50
 $EndSheet
-NoConn ~ 9850 5400
+Wire Notes Line width 12 style solid
+	5100 1400 5100 2900
+$Sheet
+S 7750 1000 1300 1900
+U 5DC1F176
+F0 "MCU" 50
+F1 "MCU.sch" 50
+F2 "SLOOP1_IN" I R 9050 1100 50
+F3 "SLOOP1_OUT" I R 9050 1200 50
+F4 "AIRS+" I R 9050 1400 50
+F5 "AIRS-" I R 9050 1500 50
+F6 "CHRG_EN" I L 7750 1550 50
+F7 "CHRG_CURRENT" I L 7750 1750 50
+F8 "SDA_GLV" I L 7750 1900 50
+F9 "SCL_GLV" I L 7750 2000 50
+F10 "~CHRG_DETECT" I L 7750 1650 50
+F11 "CAN_H" I R 9050 1600 50
+F12 "CAN_L" I R 9050 1700 50
+F13 "LV_5V" I L 7750 1200 50
+F14 "LV_RTN" I L 7750 1400 50
+F15 "BTN_LEFT" I L 7750 2150 50
+F16 "BTN_RIGHT" I L 7750 2250 50
+F17 "BTN_UP" I L 7750 2350 50
+F18 "BTN_DOWN" I L 7750 2450 50
+F19 "BTN_CENTER" I L 7750 2550 50
+F20 "DISP_MOSI" I R 9050 2450 50
+F21 "DISP_CLK" I R 9050 2350 50
+F22 "DISP_CS" I R 9050 2250 50
+F23 "DISP_DC" I R 9050 2150 50
+F24 "DISP_RST" I R 9050 2050 50
+F25 "TS_ACTIVE" I R 9050 1950 50
+F26 "CAN_SHIELD" I R 9050 1800 50
+F27 "LV_3V3" I L 7750 1300 50
+F28 "SLOOP2" I R 9050 1300 50
+F29 "RST_GLV_SEG+" I L 7750 2700 50
+F30 "RST_GLV_SEG-" I L 7750 2800 50
+F31 "LV_24V" I L 7750 1100 50
+F32 "GLV_24V" I R 9050 2600 50
+F33 "GLV_RTN" I R 9050 2700 50
+$EndSheet
+Wire Notes Line width 12 style solid
+	5100 500  5100 1300
 $EndSCHEMATC
